File: Delibird.kicad_pcb (KiCad board)
At the start: 2 copper layers, 38.1 x 25.4 mm, 26 parts, among them J2 Conn_01x04_Male, U1 ATmega16M1-AU, U2 TJA1051T, U3 NCP1117-5V, U4 NCP1117-3.3V, Y1 Crystal

Commit message: Update Delibird.kicad_pcb
Parts:
- added C9: 100n, Capacitor_SMD:C_0805_2012Metric_Pad1.15x1.40mm_HandSolder, B.Cu at (37.0, 20.7)
- added R2: 120, Resistor_SMD:R_0805_2012Metric_Pad1.15x1.40mm_HandSolder, B.Cu at (48.0, 24.8)
- renumbered ICSP to J1, GND to TP0, MISO to TP1, MOSI to TP2, SCK to TP3, 5V to TP4, 3V3 to TP5, AMP1- to TP6, AMP1+ to TP7, ADC2 to TP8
Routing:
- net +5V: track 57.7 -> 62.3 mm
- net CANH: track 4.45 -> 6.97 mm
- net CANL: track 4.44 -> 6.94 mm
