File: Laser_Stripe_Sensor/Laser_Stripe_Sensor.sch (KiCad schematic (older format))
At the start: 33 parts, among them J1 ISP-6, J1 SDRR1_Header, J2 Conn_01x04_Male, J2 SDRR1_Header, P1 Power, P2 Analog, P3 Digital, P4 Digital, U1 ATmega16M1-AU, U2 TJA1051T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

Commit message: Added IMU, and assigned footprint
Parts:
- added C10, C9: 0.1uF, Capacitor_SMD:C_0805_2012Metric_Pad1.15x1.40mm_HandSolder, symbol Device:C
- added P10: Header4, Connector_PinHeader_2.54mm:PinHeader_1x04_P2.54mm_Vertical, symbol IMU:Header4
- added P8: Header4, Connector_PinSocket_2.54mm:PinSocket_1x04_P2.54mm_Vertical, symbol IMU:Header4
- added P9: Header3, Connector_PinSocket_2.54mm:PinSocket_1x03_P2.54mm_Vertical, symbol IMU:Header3
- J1: footprint (none) -> Connector_PinHeader_2.54mm:PinHeader_2x03_P2.54mm_Vertical
- J3: renamed from J1; footprint (none) -> Connector_PinSocket_2.54mm:PinSocket_1x05_P2.54mm_Vertical; symbol Laser_Stripe_Sensor-rescue:SDRR1_Header-SDRR1 -> Laser_Stripe_Sensor-rescue:SDRR1_Header-SDRR1-Laser_Stripe_Sensor-rescue
- J4: renamed from J2; footprint (none) -> Connector_PinSocket_2.54mm:PinSocket_1x05_P2.54mm_Vertical; symbol Laser_Stripe_Sensor-rescue:SDRR1_Header-SDRR1 -> Laser_Stripe_Sensor-rescue:SDRR1_Header-SDRR1-Laser_Stripe_Sensor-rescue
- R2, R3: footprint (none) -> Resistor_SMD:R_0805_2012Metric_Pad1.15x1.40mm_HandSolder
Connections:
- net +3V3: now also C10.1, C9.1, P8.3
- net GND: now also C10.2, C9.2, P10.1, P8.4, P9.1, P9.2, P9.3
- net SCK: now also P8.1
- net DOut1: now reaches P4.4 (Pin_4)
- net DOut1: now also J3.2 (NPN(OUT)), R2.1, U1.16 (PB2)
- net DOut2: now reaches P4.6 (Pin_6)
- net DOut2: now also J4.2 (NPN(OUT)), R3.1, U1.26 (PB5)
- net CS: now reaches U1.3 (PC1)
- net CS: now also P10.2
- removed net AOut1: J3.2 (NPN(OUT)), P2.2 (Pin_2), R2.1, U1.16 (PB2)
- removed net AOut2: J4.2 (NPN(OUT)), P2.3 (Pin_3), R3.1, U1.26 (PB5)
- net MISO renamed SDO-MISO
- net MOSI renamed SDI-MOSI
- net SDI-MOSI: now also P8.2
- new net: P10.3, P10.4
Other:
- note removed: "18/01/2020"
- moved on the sheet: J2, J3, J4, P1, P2, P3, P4, R2, R3, TP0
