File: Psyduck/Psyduck.kicad_pcb (KiCad board)
At the start: 2 copper layers, 38.1 x 25.4 mm, 20 parts, among them J1 ISP-6, J2 Conn_01x04_Male, J3 Conn_01x03_Male, U1 ATmega16M1-AU, U2 TJA1051T, U3 NCP1117-5V, Y1 Crystal

Commit message: Updated shematic and layout to accomodate changes from first round of testing
Parts:
- removed R2: 120, Resistor_SMD:R_0805_2012Metric_Pad1.15x1.40mm_HandSolder
- C5, C6: value 20p -> 10p
- moved J3 2.84 mm to (17.8, 27.9)
Connections:
- J1 pad 2: +5V -> UIN
Routing:
- net UIN: track 6.57 -> 36.5 mm, vias 0 -> 1
- net +5V: track 81.8 -> 74.3 mm
- net OUTPUT+: track 23.8 -> 20.7 mm
- net CANH: track 6.97 -> 4.45 mm
- net CANL: track 6.94 -> 4.44 mm
- net Earth: vias 17 -> 5
