File: Brake_Actuator/BrakeActuator.kicad_pcb (KiCad board)
At the start: 2 copper layers, 38.1 x 25.4 mm, 27 parts, among them J1 ISP-6, J2 Conn_01x04_Male, J3 24V Connector, J4 Brake, Q1 STP55NF06L, U1 ATmega16M1-AU, U2 TJA1051T, U3 NCP1117-5V, U4 NCP1117-3.3V, Y1 Crystal

Commit message: most recent changes to brake actuator
Parts:
- added R5: 50 mili, Resistor_SMD:R_2512_6332Metric_Pad1.52x3.35mm_HandSolder, F.Cu at (63.2, 28.2)
- added TP1: TestPoint, TestPoint:TestPoint_Pad_D1.0mm, F.Cu at (69.3, 27.3)
- added TP2: TestPoint, TestPoint:TestPoint_Pad_D1.0mm, F.Cu at (66.1, 32.2)
- added TP3: TestPoint, TestPoint:TestPoint_Pad_D1.0mm, F.Cu at (69.3, 30.3)
- added TP6: TestPoint, TestPoint:TestPoint_Pad_D1.0mm, F.Cu at (72.3, 27.3)
- added TP7: TestPoint, TestPoint:TestPoint_Pad_D1.0mm, F.Cu at (69.1, 33.4)
- added TP8: TestPoint, TestPoint:TestPoint_Pad_D1.0mm, F.Cu at (72.3, 30.3)
- added U5: Sensor_Current_TSC888, Package_TO_SOT_SMD:SOT-23-5_HandSoldering, F.Cu at (61.6, 33.0)
Connections:
- Q1 pad 1: Brake+ -> Net-(Q1-Pad1)
- Q1 pad 2: Brake+ -> Net-(Q1-Pad1)
- Q1 pad 3: Brake+ -> Net-(Q1-Pad1)

Commit message: completed part for brake actuator board
Parts:
- removed TP1, TP2, TP3, TP6, TP7, TP8: TestPoint, TestPoint:TestPoint_Pad_D1.0mm
- R4, R5, U5: moved to B.Cu
- moved R4 35.4 mm to (25.9, 25.1)
- moved U5 28.8 mm to (35.8, 20.2)
- moved R5 28.6 mm to (37.4, 16.0)
- moved U2 0.51 mm to (39.4, 24.8)
- moved R2 0.26 mm to (24.4, 27.0)
Connections:
- U1 pad 13: /ADC2 -> TSCout
Routing:
- net Brake+: track 17.1 -> 52.8 mm
- net Net-(Q1-Pad1): track 0.00 -> 31.4 mm, vias 0 -> 1
- net Earth: track 12.6 -> 19.6 mm, vias 19 -> 13
- net +5V: track 57.7 -> 62.0 mm
- net TSCout: track 0.00 -> 2.75 mm, vias 0 -> 1
- net OUT: track 7.59 -> 10.1 mm
