File: Optical Ring Encoder/Optical Ring Encoder.sch (KiCad schematic (older format))
At the start: 20 parts

Commit message: Add files via upload
Parts:
- removed C?: 100n, symbol Device:C
- removed C?: 20p, symbol Device:C
- removed C?: 100p, symbol Device:C
- removed J?: ISP-6, symbol Connector:AVR-ISP-6
- removed J?: Conn_01x04_Male, symbol Connector:Conn_01x04_Male
- removed R?: 10k, symbol Device:R
- removed R?: 1k, symbol Device:R
- removed SW?: SW_Push, symbol Switch:SW_Push
- removed U?: NCP1117-3.3V, Package_TO_SOT_SMD:SOT-223-3_TabPin2, symbol Regulator_Linear:NCP1117-3.3_SOT223
- added C1, C5, C7, C8: 100n, Capacitor_SMD:C_0805_2012Metric_Pad1.15x1.40mm_HandSolder, symbol Device:C
- added C2: 100p, Capacitor_SMD:C_0805_2012Metric_Pad1.15x1.40mm_HandSolder, symbol Device:C
- added C3: 10p, Capacitor_SMD:C_0805_2012Metric_Pad1.15x1.40mm_HandSolder, symbol Device:C
- added C6, C9: 100u, Capacitor_SMD:CP_Elec_8x6.2, symbol Device:CP
- added C9: 100p, Capacitor_SMD:CP_Elec_8x6.2, symbol Device:CP
- added J1: ISP-6, Connector_PinHeader_2.54mm:PinHeader_2x03_P2.54mm_Vertical, symbol Connector:AVR-ISP-6
- added J2: Conn_01x04_Male, Connector_JST:JST_XH_S4B-XH-A-1_1x04_P2.50mm_Horizontal, symbol Connector:Conn_01x04_Male
- added R1: 10k, Resistor_SMD:R_0805_2012Metric_Pad1.15x1.40mm_HandSolder, symbol Device:R
- added TP1, TP10, TP11, TP2, TP3, TP4, TP5, TP6, TP7, TP8, TP9: TestPoint, TestPoint:TestPoint_Pad_D1.0mm, symbol Connector:TestPoint
- added U4: NCP1117-3.3V, Package_TO_SOT_SMD:SOT-223-3_TabPin2, symbol Regulator_Linear:NCP1117-3.3_SOT223
- C4: renamed from C?; value 20p -> 10p; footprint (none) -> Capacitor_SMD:C_0805_2012Metric_Pad1.15x1.40mm_HandSolder
- R3, R5: renamed from R?; footprint (none) -> RT0402FRE0780RL:RESC1005X35N
- R4, R6: renamed from R?; footprint (none) -> RMCF0201FT4K70:RESC0603X26N
- U5, U6: renamed from U?; footprint (none) -> Sensor_Optical:OPB733TR; symbol Components:OPB733TR -> Optical-Ring-Encoder-rescue:OPB733TR-Components
- Y1: renamed from Y?; footprint (none) -> Crystal:Crystal_SMD_MicroCrystal_CC8V-T1A-2Pin_2.0x1.2mm
- gave numbers to parts that had none: 3
Connections:
- net labels added: +3V3, +5V, ADC2, AMP1+, AMP1-, CANRX, CANTX, Earth, MISO_A, MOSI_A, RESET, SCK_A, UIN, XTAL1, XTAL2
- net labels removed: 5V, 5V_IN
- wire segments 81 -> 110
Other:
- note added: "4"
- moved on the sheet: C4, U1, U2, U3, Y1
